Commit message: Fix URDF xacro include for ROS 2 Jazzy
Removed ROS 1 /urdf/common_properties.xacro
include and defined material colors (black, dark, light_black) inline.

File: urdf/turtlebot3_burger_high_traction.urdf.xacro (robot description, xacro)
@@ -1,5 +1,13 @@
 <?xml version="1.0" ?>
 <robot name="turtlebot3_burger_for_autorace_2020" xmlns:xacro="http://ros.org/wiki/xacro">
-  <xacro:include filename="$(find turtlebot3_description)/urdf/common_properties.xacro"/>
+  <material name="black">
+    <color rgba="0.0 0.0 0.0 1.0"/>
+  </material>
+  <material name="dark">
+    <color rgba="0.3 0.3 0.3 1.0"/>
+  </material>
+  <material name="light_black">
+    <color rgba="0.4 0.4 0.4 1.0"/>
+  </material>
   <xacro:include filename="$(find lane_detector)/urdf/turtlebot3_burger_high_traction.gazebo.xacro"/>
   <link name="base_footprint"/>
